Commit message: test success

File: urdf/robot1_base_04.xacro (robot description, xacro)
@@ -8,4 +8,5 @@
 	<xacro:property name="radius_wheel" value="0.05" />
 	<xacro:property name="camera_link" value="0.05" />
+  <xacro:property name="M_PI" value="3.1415926535897931" />
 	<xacro:macro name="default_inertial" params="mass">
                <inertial>
@@ -16,4 +17,5 @@
                </inertial>
 	</xacro:macro>
+  <xacro:include filename="saturn_property.urdf.xacro" />
 	<link name="base_footprint">
    		<visual>
@@ -25,5 +27,5 @@
 		<!--<xacro:default_inertial mass="0.0001"/>-->
  	</link>
- 	<xacro:include filename="$(find robot1_description)/urdf/robot.gazebo" />
+ 	<xacro:include filename="robot1.gazebo" />
 	<gazebo reference="base_footprint">
 		<material>Gazebo/Green</material>
@@ -52,5 +54,5 @@
 		<xacro:default_inertial mass="10"/>
  	</link>
- 	<link name="wheel_1">
+ 	<link name="wheel_left">
    		<visual>
      			<geometry>
@@ -70,5 +72,5 @@
 		<xacro:default_inertial mass="1"/>
  	</link>
- 	<link name="wheel_2">
+ 	<link name="wheel_right">
    		<visual>
      			<geometry>
@@ -86,8 +88,8 @@
 		<xacro:default_inertial mass="1"/>
  	</link>
- 	<link name="wheel_3">
+ 	<link name="caster_wheel">
    		<visual>
      			<geometry>
-       				<cylinder length="${length_wheel}" radius="${radius_wheel}"/>
+       				<sphere radius="${radius_wheel}"/>
      			</geometry>
 			<!-- <origin rpy="0 1.5 0" xyz="0.1 -0.1 0"/> -->
@@ -97,121 +99,104 @@
 		<collision>
 			<geometry>
-       				<cylinder length="${length_wheel}" radius="${radius_wheel}"/>
+       				<sphere radius="${radius_wheel}"/>
 			</geometry>
 		</collision>
 		<xacro:default_inertial mass="1"/>
  	</link>
- 	<link name="wheel_4">
-   		<visual>
-     			<geometry>
-       				<cylinder length="${length_wheel}" radius="${radius_wheel}"/>
-     			</geometry>
-		<!--	<origin rpy="0 1.5 0" xyz="-0.1 -0.1 0"/> -->
-			<origin rpy="0 0 0" xyz="0 0 0" />
-   			<material name="black"/>
-   		</visual>
-		<collision>
-			<geometry>
-       				<cylinder length="${length_wheel}" radius="${radius_wheel}"/>
-			</geometry>
-		</collision>
-		<xacro:default_inertial mass="1"/>
- 	</link>
- <joint name="base_to_wheel1" type="continuous">
+ <joint name="base_to_wheel_left" type="continuous">
    <parent link="base_link"/>
-   <child link="wheel_1"/>
-   <origin rpy="-1.5707 0 0" xyz="0.1 0.15 0"/>
+   <child link="wheel_left"/>
+   <origin rpy="-1.5707 0 0" xyz="-0.1 0.15 0"/>
    <axis xyz="0 0 1" />
  </joint>
- <joint name="base_to_wheel2" type="continuous">
+ <joint name="base_to_wheel_right" type="continuous">
    <axis xyz="0 0 1" />
    <anchor xyz="0 0 0" />
    <limit effort="100" velocity="100" />
    <parent link="base_link"/>
-   <child link="wheel_2"/>
-   <origin rpy="-1.5707 0 0" xyz="-0.1 0.15 0"/>
+   <child link="wheel_right"/>
+   <origin rpy="-1.5707 0 0" xyz="-0.1 -0.15 0"/>
 </joint>
- <joint name="base_to_wheel3" type="continuous">
+ <joint name="base_to_caster_wheel" type="continuous">
    <parent link="base_link"/>
    <axis xyz="0 0 1" />
-   <child link="wheel_3"/>
-   <origin rpy="-1.5707 0 0" xyz="0.1 -0.15 0"/>
+   <child link="caster_wheel"/>
+   <origin rpy="-1.5707 0 0" xyz="0.1 0 0"/>
  </joint>
- <joint name="base_to_wheel4" type="continuous">
-   <parent link="base_link"/>
-   <axis xyz="0 0 1" />
-   <child link="wheel_4"/>
-   <origin rpy="-1.5707 0 0" xyz="-0.1 -0.15 0"/>
- </joint>
-  <!-- Camera joint -->
+  <!-- Camera joint
   <joint name="camera_joint" type="fixed">
     <axis xyz="0 1 0" />
-    <origin xyz="0.125 0 0.125" rpy="0 0 0"/>
+    <origin xyz="-0.1 0 0.25" rpy="0 0 0"/>
     <parent link="base_link"/>
     <child link="camera_link"/>
-  </joint>
+  </joint>-->
   <!-- Camera -->
-  <link name="camera_link">
-    <collision>
-      <origin xyz="0 0 0" rpy="0 0 0"/>
-      <geometry>
-	<box size="0.05 0.05 0.05"/>
-      </geometry>
-    </collision>
-    <visual>
-      <origin xyz="0 0 0" rpy="0 0 0"/>
-      <geometry>
-	<box size="0.05 0.05 0.05"/>
-      </geometry>
-      <material name="red">
-	<color rgba="1 0 0 1"/>
-      </material>
-    </visual>
-    <inertial>
-      <mass value="1e-5" />
-      <origin xyz="0 0 0" rpy="0 0 0"/>
-      <inertia ixx="1e-6" ixy="0" ixz="0" iyy="1e-6" iyz="0" izz="1e-6" />
-    </inertial>
-  </link>
-  <!-- Hokuyo joint -->
-  <joint name="hokuyo_joint" type="fixed">
-    <origin xyz="0.125 0.05 0.125" rpy="0 0 0"/>
-    <parent link="base_link"/>
-    <axis xyz="0 1 0" />
-    <child link="hokuyo_link"/>
-  </joint>
-  <!-- Hokuyo Laser -->
-  <link name="hokuyo_link">
-    <collision>
-      <origin xyz="0 0 0" rpy="0 0 0"/>
-      <geometry>
-	<box size="0.1 0.1 0.1"/>
-      </geometry>
-    </collision>
-    <visual>
-      <origin xyz="0 0 0" rpy="0 0 0"/>
-      <geometry>
-        <mesh filename="package://robot1_description/meshes/hokuyo.dae"/>
-      </geometry>
-    </visual>
-    <inertial>
-      <mass value="1e-5" />
-      <origin xyz="0 0 0" rpy="0 0 0"/>
-      <inertia ixx="1e-6" ixy="0" ixz="0" iyy="1e-6" iyz="0" izz="1e-6" />
-    </inertial>
-  </link>
+  <xacro:property name="kinect_cam_py" value="-0.0125"/>
+  <!-- Parameterised in part by the values in turtlebot_properties.urdf.xacro -->
+  <xacro:macro name="sensor_kinect" params="parent" />
+    <joint name="camera_rgb_joint" type="fixed">
+      <origin xyz="${cam_px} ${kinect_cam_py} ${cam_pz}" rpy="${cam_or} ${cam_op} ${cam_oy}"/>
+      <parent link="base_link"/>
+      <child link="camera_rgb_frame" />
+    </joint>
+    <link name="camera_rgb_frame"/>
+    <joint name="camera_rgb_optical_joint" type="fixed">
+      <origin xyz="0 0 0" rpy="${-M_PI/2} 0 ${-M_PI/2}" />
+      <parent link="camera_rgb_frame" />
+      <child link="camera_rgb_optical_frame" />
+    </joint>
+    <link name="camera_rgb_optical_frame"/>
+    <joint name="camera_joint" type="fixed">
+      <origin xyz="-0.031 ${-kinect_cam_py} -0.016" rpy="0 0 0"/>
+      <parent link="camera_rgb_frame"/>
+      <child link="camera_link"/>
+    </joint>
+      <link name="camera_link">
+      <visual>
+       <origin xyz="0 0 0" rpy="0 0 ${M_PI/2}"/>
+        <geometry>
+         <mesh filename="package://turtlebot_description/meshes/sensors/kinect.dae"/>
+        </geometry>
+      </visual>
+  	  <collision>
+        <origin xyz="0.0 0.0 0.0" rpy="0 0 0"/>
+  	    <geometry>
+  	      <box size="0.07271 0.27794 0.073"/>
+  	    </geometry>
+  	  </collision>
+      <inertial>
+        <mass value="0.564" />
+        <origin xyz="0 0 0" />
+        <inertia ixx="0.003881243" ixy="0.0" ixz="0.0"
+                 iyy="0.000498940" iyz="0.0"
+                 izz="0.003879257" />
+      </inertial>
+    </link>
+    <!-- The fixed joints & links below are usually published by static_transformers launched by the OpenNi launch
+         files. However, for Gazebo simulation we need them, so we add them here.
+         (Hence, don't publish them additionally!) -->
+	<joint name="camera_depth_joint" type="fixed">
+	  <origin xyz="0 ${2 * -kinect_cam_py} 0" rpy="0 0 0" />
+	  <parent link="camera_rgb_frame" />
+	  <child link="camera_depth_frame" />
+	</joint>
+	<link name="camera_depth_frame"/>
+	<joint name="camera_depth_optical_joint" type="fixed">
+	  <origin xyz="0 0 0" rpy="${-M_PI/2} 0 ${-M_PI/2}" />
+	  <parent link="camera_depth_frame" />
+	  <child link="camera_depth_optical_frame" />
+	</joint>
+	<link name="camera_depth_optical_frame"/>
   <!-- Drive controller -->
 <gazebo>
-  <plugin name="skid_steer_drive_controller" filename="libgazebo_ros_skid_steer_drive.so">
+  <plugin name="differential_drive_controller" filename="libgazebo_ros_diff_drive.so">
     <updateRate>100.0</updateRate>
     <robotNamespace>/</robotNamespace>
-    <leftFrontJoint>base_to_wheel1</leftFrontJoint>
-    <rightFrontJoint>base_to_wheel3</rightFrontJoint>
-    <leftRearJoint>base_to_wheel2</leftRearJoint>
-    <rightRearJoint>base_to_wheel4</rightRearJoint>
+    <leftJoint>base_to_wheel_left</leftJoint>
+    <rightJoint>base_to_wheel_right</rightJoint>
     <wheelSeparation>4</wheelSeparation>
     <wheelDiameter>0.1</wheelDiameter>
     <robotBaseFrame>base_footprint</robotBaseFrame>
-    <torque>1</torque>
+    <wheelTorque>5</wheelTorque>
     <topicName>cmd_vel</topicName>
     <commandTopic>cmd_vel</commandTopic>

Commit message: make camera_link parent

File: urdf/robot1_base_04.xacro (robot description, xacro)
@@ -135,10 +135,9 @@
   <!-- Parameterised in part by the values in turtlebot_properties.urdf.xacro -->
   <xacro:macro name="sensor_kinect" params="parent" />
-    <joint name="camera_rgb_joint" type="fixed">
+    <joint name="camera_joint" type="fixed">
       <origin xyz="${cam_px} ${kinect_cam_py} ${cam_pz}" rpy="${cam_or} ${cam_op} ${cam_oy}"/>
       <parent link="base_link"/>
-      <child link="camera_rgb_frame" />
+      <child link="camera_link" />
     </joint>
-    <link name="camera_rgb_frame"/>
     <joint name="camera_rgb_optical_joint" type="fixed">
       <origin xyz="0 0 0" rpy="${-M_PI/2} 0 ${-M_PI/2}" />
@@ -147,9 +146,10 @@
     </joint>
     <link name="camera_rgb_optical_frame"/>
-    <joint name="camera_joint" type="fixed">
+    <joint name="camera_rgb_joint" type="fixed">
       <origin xyz="-0.031 ${-kinect_cam_py} -0.016" rpy="0 0 0"/>
-      <parent link="camera_rgb_frame"/>
-      <child link="camera_link"/>
+      <parent link="camera_link"/>
+      <child link="camera_rgb_frame"/>
     </joint>
+    <link name="camera_rgb_frame"/>
       <link name="camera_link">
       <visual>
@@ -178,5 +178,5 @@
 	<joint name="camera_depth_joint" type="fixed">
 	  <origin xyz="0 ${2 * -kinect_cam_py} 0" rpy="0 0 0" />
-	  <parent link="camera_rgb_frame" />
+	  <parent link="camera_link" />
 	  <child link="camera_depth_frame" />
 	</joint>
